File: ergo60tilt/ergo60tilt.kicad_pcb (KiCad board)
At the start: 2 copper layers, 141 parts, among them J1 Conn_01x03, K0 KEYSW, K1 KEYSW, K2 KEYSW, K3 KEYSW, K4 KEYSW, K5 KEYSW, K6 KEYSW, K7 KEYSW, K8 KEYSW, K9 KEYSW, SW1 SW_PUSH, U1 ProMicro

Commit message: push rotated pcb
Parts:
- KRBrc1: moved to F.Cu
- moved D62 232.2 mm to (328.6, 94.3), turned to 190 degrees
- moved D61 212.4 mm to (303.3, 98.1), turned to 190 degrees
- moved D49 196.2 mm to (278.0, 105.6), turned to 190 degrees
- moved D60 193.7 mm to (301.3, 62.8), turned to 190 degrees
- moved D66 182.0 mm to (274.1, 87.0), turned to 190 degrees
- moved D54 180.1 mm to (257.8, 104.3), turned to 190 degrees
- moved D59 179.0 mm to (292.7, 45.0), turned to 190 degrees
- moved D58 172.9 mm to (292.3, 25.7), turned to 190 degrees
- moved D65 169.1 mm to (270.8, 68.2), turned to 190 degrees
- moved H3 169.1 mm to (172.6, 141.7)
- moved H4 165.7 mm to (162.5, 136.9)
- moved D53 165.4 mm to (254.5, 85.6), turned to 190 degrees
- moved D41 165.1 mm to (238.2, 103.0), turned to 190 degrees
- moved H1 164.6 mm to (155.4, 141.7)
- moved D46 159.6 mm to (220.3, 111.0), turned to 190 degrees
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
Commit message: push completed orgonati. update readme
Parts:
- removed J1: Conn_01x03, Pin_Headers:Pin_Header_Angled_1x03_Pitch1.00mm
- added JGND1: Conn_01x01, Connectors:Pin_d0.9mm_L10.0mm_W2.4mm_FlatFork, B.Cu at (146.8, 41.7)
- added JRGB1: Conn_01x01, Connectors:Pin_d0.9mm_L10.0mm_W2.4mm_FlatFork, B.Cu at (146.8, 35.6)
- added JVCC1: Conn_01x01, Connectors:Pin_d0.9mm_L10.0mm_W2.4mm_FlatFork, B.Cu at (146.8, 38.6)
- moved H5 177.9 mm to (21.4, 40.5)
- moved H6 175.4 mm to (307.2, 40.5)
- moved H3 125.8 mm to (292.9, 104.8)
- moved H1 125.2 mm to (35.7, 104.8)
- moved H2 63.5 mm to (164.3, 71.4)
- moved H4 13.2 mm to (164.3, 150.0)
- moved D39 7.75 mm to (179.1, 134.6), turned to 105 degrees
- moved D33 7.70 mm to (149.0, 134.5), turned to 75 degrees
- moved KSpace1 6.93 mm to (140.0, 131.8), turned to 75 degrees
- moved KEnt1 6.93 mm to (188.6, 131.7), turned to 285 degrees
- moved D37 6.86 mm to (173.6, 77.5), turned to 195 degrees
- moved D1 6.82 mm to (31.8, 19.9), turned to 165 degrees
- moved D31 6.81 mm to (154.4, 77.4), turned to 165 degrees
- moved D62 6.74 mm to (329.2, 87.6), turned to 195 degrees
- moved KRBrc1 6.61 mm to (176.3, 85.7), turned to 15 degrees
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Routing:
- net /row0: track 0.00 -> 597.9 mm, vias 0 -> 16
- net /row5: track 0.00 -> 551.3 mm, vias 0 -> 27
- net /row1: track 0.00 -> 532.9 mm
- net /row6: track 0.00 -> 506.9 mm, vias 0 -> 35
- net /row2: track 0.00 -> 488.0 mm, vias 0 -> 12
- net /row4: track 0.00 -> 407.8 mm, vias 0 -> 4
- net /row3: track 0.00 -> 372.4 mm, vias 0 -> 9
- net /col7: track 0.00 -> 303.2 mm
- net /row8: track 0.00 -> 299.4 mm, vias 0 -> 19
- net /col0: track 0.00 -> 296.7 mm
- net /col1: track 0.00 -> 274.6 mm
- net /row7: track 0.00 -> 263.2 mm, vias 0 -> 17
- net /col6: track 0.00 -> 236.4 mm
- net /col2: track 0.00 -> 197.4 mm
- net /col5: track 0.00 -> 191.3 mm
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- added copper zone on F.Cu, net GND
Other:
- board outline added: 352.4 x 142.9 mm
- board text added: "OrgoNati V1 9/5/2018"
- board text added: "design by u/lizardsticks in kicad"
