File: ergo60tilt/ergo60tilt.sch (KiCad schematic (older format))
At the start: 141 parts, among them J1 Conn_01x03, K0 KEYSW, K1 KEYSW, K2 KEYSW, K3 KEYSW, K4 KEYSW, K5 KEYSW, K6 KEYSW, K7 KEYSW, K8 KEYSW, K9 KEYSW, SW1 SW_PUSH, U1 ProMicro

Commit message: push completed orgonati. update readme
Parts:
- removed J1: Conn_01x03, Pin_Headers:Pin_Header_Angled_1x03_Pitch1.00mm, symbol Conn_01x03
- added JGND1, JRGB1, JVCC1: Conn_01x01, Connectors:Pin_d0.9mm_L10.0mm_W2.4mm_FlatFork, symbol Conn_01x01
Connections:
- net GND: now also JGND1.1 (Pin_1)
- net RGB: now also JRGB1.1 (Pin_1)
- net VCC: now also JVCC1.1 (Pin_1)
Changed lines of the file:
@@
 LIBS:contrib
 LIBS:valves
-LIBS:keyboard_parts
-LIBS:promicro
 LIBS:ergo60tilt-cache
 EELAYER 25 0
@@
 L GND #PWR01
 U 1 1 5B95A910
-P 2600 6500
-F 0 "#PWR01" H 2600 6250 50  0001 C CNN
-F 1 "GND" H 2600 6350 50  0000 C CNN
-F 2 "" H 2600 6500 50  0001 C CNN
-F 3 "" H 2600 6500 50  0001 C CNN
-	1    2600 6500
+P 2650 6500
+F 0 "#PWR01" H 2650 6250 50  0001 C CNN
+F 1 "GND" H 2650 6350 50  0000 C CNN
+F 2 "" H 2650 6500 50  0001 C CNN
+F 3 "" H 2650 6500 50  0001 C CNN
+	1    2650 6500
 	0    -1   -1   0
 $EndComp
@@
 	2700 6600 2400 6600
 Wire Wire Line
-	2600 6500 2400 6500
+	2400 6500 2650 6500
 Wire Wire Line
 	2400 6700 2600 6700
@@
 	1    0    0    -1
 $EndComp
-$Comp
-L Conn_01x03 J1
-U 1 1 5B980126
-P 4800 6900
-F 0 "J1" H 4800 7100 50  0000 C CNN
-F 1 "Conn_01x03" H 4800 6700 50  0000 C CNN
-F 2 "Pin_Headers:Pin_Header_Angled_1x03_Pitch1.00mm" H 4800 6900 50  0001 C CNN
-F 3 "" H 4800 6900 50  0001 C CNN
-	1    4800 6900
-	1    0    0    -1
-$EndComp
-Text Label 4600 6800 2    60   ~ 0
+Text Label 4200 6650 2    60   ~ 0
 RGB
 $Comp
 L VCC #PWR05
 U 1 1 5B980AB3
-P 4500 6900
-F 0 "#PWR05" H 4500 6750 50  0001 C CNN
-F 1 "VCC" H 4500 7050 50  0000 C CNN
-F 2 "" H 4500 6900 50  0001 C CNN
-F 3 "" H 4500 6900 50  0001 C CNN
-	1    4500 6900
+P 4150 6950
+F 0 "#PWR05" H 4150 6800 50  0001 C CNN
+F 1 "VCC" H 4150 7100 50  0000 C CNN
+F 2 "" H 4150 6950 50  0001 C CNN
+F 3 "" H 4150 6950 50  0001 C CNN
+	1    4150 6950
 	0    -1   -1   0
 $EndComp
@@
 L GND #PWR06
 U 1 1 5B980BE1
-P 4350 7000
-F 0 "#PWR06" H 4350 6750 50  0001 C CNN
-F 1 "GND" H 4350 6850 50  0000 C CNN
-F 2 "" H 4350 7000 50  0001 C CNN
-F 3 "" H 4350 7000 50  0001 C CNN
-	1    4350 7000
+P 4200 7300
+F 0 "#PWR06" H 4200 7050 50  0001 C CNN
+F 1 "GND" H 4200 7150 50  0000 C CNN
+F 2 "" H 4200 7300 50  0001 C CNN
+F 3 "" H 4200 7300 50  0001 C CNN
+	1    4200 7300
 	0    1    1    0
 $EndComp
-Wire Wire Line
-	4500 6900 4600 6900
-Wire Wire Line
-	4600 7000 4350 7000
+$Comp
+L Conn_01x01 JVCC1
+U 1 1 5B90CBBB
+P 4400 6950
+F 0 "JVCC1" H 4400 7050 50  0000 C CNN
+F 1 "Conn_01x01" H 4400 6850 50  0000 C CNN
+F 2 "Connectors:Pin_d0.9mm_L10.0mm_W2.4mm_FlatFork" H 4400 6950 50  0001 C CNN
+F 3 "" H 4400 6950 50  0001 C CNN
+	1    4400 6950
+	1    0    0    -1
+$EndComp
+$Comp
+L Conn_01x01 JGND1
+U 1 1 5B90CDC8
+P 4400 7300
+F 0 "JGND1" H 4400 7400 50  0000 C CNN
+F 1 "Conn_01x01" H 4400 7200 50  0000 C CNN
+F 2 "Connectors:Pin_d0.9mm_L10.0mm_W2.4mm_FlatFork" H 4400 7300 50  0001 C CNN
+F 3 "" H 4400 7300 50  0001 C CNN
+	1    4400 7300
+	1    0    0    -1
+$EndComp
+$Comp
+L Conn_01x01 JRGB1
+U 1 1 5B90CF93
+P 4400 6650
+F 0 "JRGB1" H 4400 6750 50  0000 C CNN
+F 1 "Conn_01x01" H 4400 6550 50  0000 C CNN
+F 2 "Connectors:Pin_d0.9mm_L10.0mm_W2.4mm_FlatFork" H 4400 6650 50  0001 C CNN
+F 3 "" H 4400 6650 50  0001 C CNN
+	1    4400 6650
+	1    0    0    -1
+$EndComp
+Wire Wire Line
+	4150 6950 4200 6950
 $EndSCHEMATC
